File: pcb/hackpad.kicad_pcb (KiCad board)
At the start: 2 copper layers, 41 x 62.5 mm, 7 parts, among them SW1 SW_Push, SW2 SW_Push, SW3 SW_Push, SW4 SW_Push, U1 XIAO-RP2040-DIP

Commit message: Made the thing actually unique and cool and stuff
yay!
Parts:
- added G***: LOGO, LOGO, F.Cu at (206.0, 92.0)
- added G***: LOGO, LOGO, F.Cu at (158.0, 81.0)
- added G***: LOGO, LOGO, F.Cu at (200.0, 109.0)
- added G***: LOGO, LOGO, F.Cu at (161.0, 110.0)
- moved SW2 27.2 mm to (164.5, 123.9)
- moved SW1 19.1 mm to (183.5, 104.9)
- moved SW4 19.1 mm to (202.6, 123.9)
- moved SW3 19.1 mm to (183.5, 123.9)
- moved D2 13.3 mm to (198.5, 88.0)
- moved U1 9.62 mm to (181.0, 88.0)
- moved D1 7.50 mm to (163.5, 88.0)
Routing:
- net Net-(U1-GPIO2/SCK): track 18.0 -> 56.4 mm
- net Net-(U1-GPIO4/MISO): track 56.1 -> 45.1 mm
- net Net-(U1-GPIO1/RX): track 33.2 -> 22.8 mm
- net GND: track 98.8 -> 107.0 mm
- net Net-(D1-DIN): track 6.85 -> 0.00 mm
- net +5V: track 39.5 -> 45.4 mm
- net Net-(D1-DOUT): track 48.6 -> 53.6 mm
- net Net-(U1-GPIO3/MOSI): track 46.2 -> 41.6 mm
Other:
- board size 41 x 62.5 mm -> 62 x 63 mm
- board text added: "Rohan's HackPad :3"
- board text removed: "Rohan's Macro Board :3"

Commit message: Fixed everything once again
I hope this is the last time before submitting.
Updated KMK and other KiCad stuff. Made it cooler I guess.
Parts:
- removed D2: SK6812MINI, LED_SMD:LED_SK6812MINI_PLCC4_3.5x3.5mm_P1.75mm
- removed the G*** at (206.0, 92.0)
- removed the G*** at (158.0, 81.0)
- added G***: LOGO, LOGO, F.Cu at (161.0, 82.0)
- added SW5: RotaryEncoder_Switch, Rotary_Encoder:RotaryEncoder_Alps_EC11E-Switch_Vertical_H20mm, F.Cu at (193.5, 84.0)
Connections:
- D1 pad 1: Net-(D1-DOUT) -> unconnected-(D1-DOUT-Pad1)
- D1 pad 4: +5V -> Net-(D1-VDD)
- U1 pad 1: unconnected-(U1-GPIO26/ADC0/A0-Pad1) -> Net-(U1-GPIO26/ADC0/A0)
- U1 pad 13: unconnected-(U1-GND-Pad13) -> GND
- U1 pad 14: unconnected-(U1-VBUS-Pad14) -> Net-(D1-VDD)
- U1 pad 2: unconnected-(U1-GPIO27/ADC1/A1-Pad2) -> Net-(U1-GPIO27/ADC1/A1)
- U1 pad 3: unconnected-(U1-GPIO28/ADC2/A2-Pad3) -> Net-(U1-GPIO28/ADC2/A2)
Routing:
- net Net-(D1-DOUT): track 53.6 -> 0.00 mm
- net Net-(U1-GPIO28/ADC2/A2): track 0.00 -> 45.8 mm
- net +5V: track 45.4 -> 0.00 mm
- net GND: track 107.0 -> 134.8 mm
- net Net-(D1-VDD): track 0.00 -> 26.2 mm
- net Net-(U1-GPIO26/ADC0/A0): track 0.00 -> 23.9 mm
- net Net-(U1-GPIO27/ADC1/A1): track 0.00 -> 22.6 mm
- net Net-(D1-DIN): track 0.00 -> 8.82 mm
- net Net-(U1-GPIO2/SCK): track 56.4 -> 58.0 mm
