File: pcb/hackpad.kicad_sch (KiCad schematic)
At the start: 7 parts, among them SW1 SW_Push, SW2 SW_Push, SW3 SW_Push, SW4 SW_Push, U1 XIAO-RP2040-DIP

Commit message: Made the thing actually unique and cool and stuff
yay!
Parts:
- SW1, SW2, SW3, SW4: footprint Button_Switch_Keyboard:SW_Cherry_MX_1.00u_PCB -> real_folder:MX-Solderable-1U
Changed lines of the file:
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@@
 			)
 		)
-		(property "Footprint" "Button_Switch_Keyboard:SW_Cherry_MX_1.00u_PCB"
+		(property "Footprint" "real_folder:MX-Solderable-1U"
 			(at 107.95 118.11 0)
 			(effects
@@
 			)
 		)
-		(property "Footprint" "Button_Switch_Keyboard:SW_Cherry_MX_1.00u_PCB"
+		(property "Footprint" "real_folder:MX-Solderable-1U"
 			(at 107.95 105.41 0)
 			(effects
@@
 			)
 		)
-		(property "Footprint" "Button_Switch_Keyboard:SW_Cherry_MX_1.00u_PCB"
+		(property "Footprint" "real_folder:MX-Solderable-1U"
 			(at 107.95 92.71 0)
 			(effects
@@
 			)
 		)
-		(property "Footprint" "Button_Switch_Keyboard:SW_Cherry_MX_1.00u_PCB"
+		(property "Footprint" "real_folder:MX-Solderable-1U"
 			(at 107.95 130.81 0)
 			(effects

Commit message: Fixed everything once again
I hope this is the last time before submitting.
Updated KMK and other KiCad stuff. Made it cooler I guess.
Parts:
- removed D2: SK6812MINI, LED_SMD:LED_SK6812MINI_PLCC4_3.5x3.5mm_P1.75mm, symbol LED:SK6812MINI
- added SW5: RotaryEncoder_Switch, Rotary_Encoder:RotaryEncoder_Alps_EC11E-Switch_Vertical_H20mm, symbol Device:RotaryEncoder_Switch
Connections:
- net +5V is gone; now on an unnamed net: D1.4 (VDD)
- net GND: now also U1.13 (GND), SW5.C, SW5.S1
- net at U1.1 (GPIO26/ADC0/A0): now also SW5.A
- net at U1.2 (GPIO27/ADC1/A1): now also SW5.B
- net at U1.3 (GPIO28/ADC2/A2): now also SW5.S2
Other:
- moved on the sheet: D1, SW1, SW2, SW3, SW4, U1
